File: PCB/EC87/EC87.kicad_pcb (KiCad board)
At the start: 2 copper layers, 344 x 123.8 mm, 109 parts, among them J1 AVR-ISP-6-Connector, SW1 SW_Push, SW10 EC_SW, SW11 EC_SW, SW12 EC_SW, SW13 EC_SW, SW14 EC_SW, SW15 EC_SW, SW16 EC_SW, SW17 EC_SW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

Commit message: WIP
Routing:
- net ROW0: track 21.3 -> 494.3 mm, vias 16 -> 32
- net ROW5: track 13.7 -> 439.9 mm, vias 11 -> 22
