File: PCB/EC87/EC87.kicad_sch (KiCad schematic)
At the start: 21 parts, among them J1 AVR-ISP-6-Connector, SW1 SW_Push, U1 ATmega32U4-A, Y1 16MHz

Commit message: WIP
Connections:
- net COL0: no longer names the net of U1.41 (PF0)
- net COL1: no longer names the net of U1.40 (PF1)
- net COL2: no longer names the net of U1.39 (PF4)
- net COL3: no longer names the net of U1.38 (PF5)
- net COL4 renamed ADC
- net COL5: no longer names the net of U1.36 (PF7)
- net COL6: no longer names the net of U1.32 (PC7)
- net COL7: no longer names the net of U1.31 (PC6)
- net COL8: no longer names the net of U1.20 (PD2)
- net Caps_LED: no longer names the net of U1.22 (PD5)
- net ROW0: no longer names the net of U1.8 (PB0)
- net ROW1 renamed SCK
- net ROW10: no longer names the net of U1.26 (PD6)
- net ROW11: no longer names the net of U1.25 (PD4)
- net ROW4: no longer names the net of U1.18 (PD0)
- net ROW5: no longer names the net of U1.19 (PD1)
- net ROW6: no longer names the net of U1.29 (PB5)
- net ROW7: no longer names the net of U1.30 (PB6)
- net ROW8: no longer names the net of U1.27 (PD7)
- net ROW9: no longer names the net of U1.28 (PB4)
- net Scroll_LED: no longer names the net of U1.1 (PE6)
- no-connect marks 5 -> 3
Other:
- added sheet analog (analog.kicad_sch)
- moved on the sheet: D1, F1, J1
