File: PCB/EC87.kicad_pcb (KiCad board)
At the start: 2 copper layers, 344 x 123.8 mm, 109 parts, among them J1 AVR-ISP-6-Connector, SW1 SW_Push, SW10 EC_SW, SW11 EC_SW, SW12 EC_SW, SW13 EC_SW, SW14 EC_SW, SW15 EC_SW, SW16 EC_SW, SW17 EC_SW, SW18 EC_SW, SW19 EC_SW, SW2 EC_SW, SW20 EC_SW, SW21 EC_SW, SW22 EC_SW, SW23 EC_SW, SW24 EC_SW, SW25 EC_SW, SW26 EC_SW, SW27 EC_SW, SW28 EC_SW, SW29 EC_SW, SW3 EC_SW, SW30 EC_SW, SW31 EC_SW, SW32 EC_SW, SW33 EC_SW, SW34 EC_SW, SW35 EC_SW, SW36 EC_SW, SW37 EC_SW, SW38 EC_SW, SW39 EC_SW, SW4 EC_SW, SW40 EC_SW, SW41 EC_SW, SW42 EC_SW, SW43 EC_SW, SW44 EC_SW, SW45 EC_SW, SW46 EC_SW, SW47 EC_SW, SW48 EC_SW, SW49 EC_SW, SW5 EC_SW, SW50 EC_SW, SW51 EC_SW, SW52 EC_SW, SW53 EC_SW, SW54 EC_SW, SW55 EC_SW, SW56 EC_SW, SW57 EC_SW, SW58 EC_SW, SW59 EC_SW, SW6 EC_SW, SW60 EC_SW, SW61 EC_SW, SW62 EC_SW, SW63 EC_SW, SW64 EC_SW, SW65 EC_SW, SW66 EC_SW, SW67 EC_SW, SW68 EC_SW, SW69 EC_SW, SW7 EC_SW, SW70 EC_SW, SW71 EC_SW, SW72 EC_SW, SW73 EC_SW, SW74 EC_SW, SW75 EC_SW, SW76 EC_SW, SW77 EC_SW, SW78 EC_SW, SW79 EC_SW, SW8 EC_SW, SW80 EC_SW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

Commit message: WIP
Parts:
- moved C3 40.5 mm to (332.5, 155.8)
- moved C5 40.5 mm to (355.1, 158.1)
- moved F1 40.5 mm to (327.8, 92.6)
- moved Y1 40.5 mm to (353.2, 160.1)
- moved C1 40.5 mm to (351.6, 154.2)
- moved C4 40.5 mm to (332.5, 164.7)
- moved C6 40.5 mm to (341.3, 150.6)
- moved C7 40.5 mm to (355.4, 162.3)
- moved D1 40.5 mm to (327.8, 96.3)
- moved R5 40.5 mm to (329.6, 165.6)
- moved R6 40.5 mm to (348.7, 150.6)
- moved SW1 40.5 mm to (364.0, 160.3)
- moved R1 40.5 mm to (331.9, 92.3)
- moved R2 40.5 mm to (323.6, 92.3)
- moved R3 40.5 mm to (328.9, 103.3)
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Routing:
- net ROW0: track 494.3 -> 0.00 mm, vias 32 -> 0
- net ROW5: track 439.9 -> 0.00 mm, vias 22 -> 0
- net COL10: track 129.1 -> 0.00 mm, vias 6 -> 0
- net COL13: track 121.1 -> 0.00 mm, vias 6 -> 0
- net COL2: track 120.0 -> 0.00 mm, vias 6 -> 0
- net COL11: track 118.4 -> 0.00 mm, vias 5 -> 0
- net COL0: track 116.5 -> 0.00 mm, vias 6 -> 0
- net COL5: track 116.2 -> 0.00 mm, vias 6 -> 0
- net COL12: track 114.6 -> 0.00 mm, vias 4 -> 0
- net COL6: track 98.7 -> 0.00 mm, vias 5 -> 0
- net COL7: track 98.6 -> 0.00 mm, vias 5 -> 0
- net COL8: track 98.6 -> 0.00 mm, vias 5 -> 0
- net COL9: track 98.4 -> 0.00 mm, vias 5 -> 0
- net COL1: track 96.9 -> 0.00 mm, vias 5 -> 0
- net COL4: track 95.9 -> 0.00 mm, vias 5 -> 0
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- removed copper zone on B.Cu, net GND
Other:
- board size 344 x 123.8 mm -> 354 x 127.3 mm
- board text removed: "1.00u"
- board text removed: "1.25u"
- board text removed: "1.5u"
- board text removed: "6.25u"
- board text removed: "PCB by Cipulot"
