File: PCB/EC87.kicad_pcb (KiCad board)
At the start: 2 copper layers, 354 x 127.3 mm, 109 parts, among them J1 AVR-ISP-6-Connector, SW1 SW_Push, SW10 EC_SW, SW11 EC_SW, SW12 EC_SW, SW13 EC_SW, SW14 EC_SW, SW15 EC_SW, SW16 EC_SW, SW17 EC_SW, SW18 EC_SW, SW19 EC_SW, SW2 EC_SW, SW20 EC_SW, SW21 EC_SW, SW22 EC_SW, SW23 EC_SW, SW24 EC_SW, SW25 EC_SW, SW26 EC_SW, SW27 EC_SW, SW28 EC_SW, SW29 EC_SW, SW3 EC_SW, SW30 EC_SW, SW31 EC_SW, SW32 EC_SW, SW33 EC_SW, SW34 EC_SW, SW35 EC_SW, SW36 EC_SW, SW37 EC_SW, SW38 EC_SW, SW39 EC_SW, SW4 EC_SW, SW40 EC_SW, SW41 EC_SW, SW42 EC_SW, SW43 EC_SW, SW44 EC_SW, SW45 EC_SW, SW46 EC_SW, SW47 EC_SW, SW48 EC_SW, SW49 EC_SW, SW5 EC_SW, SW50 EC_SW, SW51 EC_SW, SW52 EC_SW, SW53 EC_SW, SW54 EC_SW, SW55 EC_SW, SW56 EC_SW, SW57 EC_SW, SW58 EC_SW, SW59 EC_SW, SW6 EC_SW, SW60 EC_SW, SW61 EC_SW, SW62 EC_SW, SW63 EC_SW, SW64 EC_SW, SW65 EC_SW, SW66 EC_SW, SW67 EC_SW, SW68 EC_SW, SW69 EC_SW, SW7 EC_SW, SW70 EC_SW, SW71 EC_SW, SW72 EC_SW, SW73 EC_SW, SW74 EC_SW, SW75 EC_SW, SW76 EC_SW, SW77 EC_SW, SW78 EC_SW, SW79 EC_SW, SW8 EC_SW, SW80 EC_SW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

Commit message: WIP
Parts:
- removed J1: AVR-ISP-6-Connector, cipulot_parts:Reset_Pretty
- removed JP2: Jumper_NC_Small, Jumper:SolderJumper-2_P1.3mm_Bridged_Pad1.0x1.5mm
- added JP1: Jumper_NC_Small, Jumper:SolderJumper-2_P1.3mm_Bridged_Pad1.0x1.5mm, F.Cu at (376.8, 172.0)
- moved C2 127.4 mm to (472.2, 153.9)
- moved AU 106.2 mm to (446.0, 142.2)
- moved C1 106.2 mm to (456.3, 136.6)
- moved C5 106.2 mm to (459.8, 140.5)
- moved C6 106.2 mm to (446.0, 133.0)
- moved C7 106.2 mm to (460.1, 144.7)
- moved MU 106.2 mm to (446.0, 142.2)
- moved R5 106.2 mm to (434.3, 148.0)
- moved R6 106.2 mm to (453.4, 133.0)
- moved C3 106.2 mm to (437.2, 138.2)
- moved C4 106.2 mm to (437.2, 147.1)
- moved SW1 106.2 mm to (468.7, 142.7)
- moved Y1 106.2 mm to (457.9, 142.5)
- turned SW24 to 180 degrees
- turned SW25 to 180 degrees
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Connections:
- SW10 pad 3: GNDA -> GND
- SW11 pad 3: GNDA -> GND
- SW12 pad 3: GNDA -> GND
- SW13 pad 3: GNDA -> GND
- SW14 pad 3: GNDA -> GND
- SW15 pad 3: GNDA -> GND
- SW16 pad 3: GNDA -> GND
- SW17 pad 3: GNDA -> GND
- SW18 pad 3: GNDA -> GND
- SW19 pad 3: GNDA -> GND
- SW2 pad 3: GNDA -> GND
- SW20 pad 3: GNDA -> GND
- SW21 pad 3: GNDA -> GND
- SW22 pad 3: GNDA -> GND
- SW23 pad 3: GNDA -> GND
- SW24 pad 3: GNDA -> GND
- SW25 pad 3: GNDA -> GND
- SW26 pad 3: GNDA -> GND
- SW27 pad 3: GNDA -> GND
- SW28 pad 3: GNDA -> GND
- SW29 pad 3: GNDA -> GND
- SW3 pad 3: GNDA -> GND
- SW30 pad 3: GNDA -> GND
- SW31 pad 3: GNDA -> GND
- SW32 pad 3: GNDA -> GND
- SW33 pad 3: GNDA -> GND
- SW34 pad 3: GNDA -> GND
- SW35 pad 2: MOSI -> ROW2
- SW35 pad 3: GNDA -> GND
- SW36 pad 2: MOSI -> ROW2
- SW36 pad 3: GNDA -> GND
- SW37 pad 2: MOSI -> ROW2
- SW37 pad 3: GNDA -> GND
- SW38 pad 2: MOSI -> ROW2
- SW38 pad 3: GNDA -> GND
- SW39 pad 2: MOSI -> ROW2
- SW39 pad 3: GNDA -> GND
- SW4 pad 3: GNDA -> GND
- SW40 pad 2: MOSI -> ROW2
- SW40 pad 3: GNDA -> GND
- SW41 pad 2: MOSI -> ROW2
- SW41 pad 3: GNDA -> GND
- SW42 pad 2: MOSI -> ROW2
- SW42 pad 3: GNDA -> GND
- SW43 pad 2: MOSI -> ROW2
- SW43 pad 3: GNDA -> GND
- SW44 pad 2: MOSI -> ROW2
- SW44 pad 3: GNDA -> GND
- SW45 pad 2: MOSI -> ROW2
- SW45 pad 3: GNDA -> GND
- SW46 pad 2: MOSI -> ROW2
- SW46 pad 3: GNDA -> GND
- SW47 pad 2: MOSI -> ROW2
- SW47 pad 3: GNDA -> GND
- SW48 pad 2: MOSI -> ROW2
- SW48 pad 3: GNDA -> GND
- SW49 pad 2: MOSI -> ROW2
- SW49 pad 3: GNDA -> GND
- SW5 pad 3: GNDA -> GND
- SW50 pad 2: MOSI -> ROW2
- SW50 pad 3: GNDA -> GND
- SW51 pad 2: MOSI -> ROW2
- SW51 pad 3: GNDA -> GND
- SW52 pad 2: MISO -> ROW3
- SW52 pad 3: GNDA -> GND
- SW53 pad 2: MISO -> ROW3
- SW53 pad 3: GNDA -> GND
- SW54 pad 2: MISO -> ROW3
- SW54 pad 3: GNDA -> GND
- SW55 pad 2: MISO -> ROW3
- SW55 pad 3: GNDA -> GND
- SW56 pad 2: MISO -> ROW3
- SW56 pad 3: GNDA -> GND
- SW57 pad 2: MISO -> ROW3
- SW57 pad 3: GNDA -> GND
- SW58 pad 2: MISO -> ROW3
- SW58 pad 3: GNDA -> GND
- SW59 pad 2: MISO -> ROW3
- SW59 pad 3: GNDA -> GND
- SW6 pad 3: GNDA -> GND
- SW60 pad 2: MISO -> ROW3
- SW60 pad 3: GNDA -> GND
- SW61 pad 2: MISO -> ROW3
- SW61 pad 3: GNDA -> GND
- SW62 pad 2: MISO -> ROW3
- SW62 pad 3: GNDA -> GND
- SW63 pad 2: MISO -> ROW3
- SW63 pad 3: GNDA -> GND
- SW64 pad 2: MISO -> ROW3
- SW64 pad 3: GNDA -> GND
- SW65 pad 3: GNDA -> GND
- SW66 pad 3: GNDA -> GND
- SW67 pad 3: GNDA -> GND
- SW68 pad 3: GNDA -> GND
- SW69 pad 3: GNDA -> GND
- SW7 pad 3: GNDA -> GND
- SW70 pad 3: GNDA -> GND
- SW71 pad 3: GNDA -> GND
- SW72 pad 3: GNDA -> GND
- SW73 pad 3: GNDA -> GND
- SW74 pad 3: GNDA -> GND
- SW75 pad 3: GNDA -> GND
- SW76 pad 3: GNDA -> GND
- SW77 pad 3: GNDA -> GND
- SW78 pad 3: GNDA -> GND
- SW79 pad 3: GNDA -> GND
- SW8 pad 3: GNDA -> GND
- SW80 pad 3: GNDA -> GND
- SW81 pad 3: GNDA -> GND
- SW82 pad 3: GNDA -> GND
- SW83 pad 3: GNDA -> GND
- SW84 pad 3: GNDA -> GND
- SW85 pad 3: GNDA -> GND
- SW86 pad 3: GNDA -> GND
- SW87 pad 3: GNDA -> GND
- SW88 pad 3: GNDA -> GND
- SW9 pad 3: GNDA -> GND
Routing:
- net COL10: track 0.00 -> 136.9 mm, vias 0 -> 6
- net COL13: track 0.00 -> 125.4 mm, vias 0 -> 6
- net COL11: track 0.00 -> 121.4 mm, vias 0 -> 5
- net COL2: track 0.00 -> 120.7 mm, vias 0 -> 6
- net COL5: track 0.00 -> 118.2 mm, vias 0 -> 6
- net COL12: track 0.00 -> 116.9 mm, vias 0 -> 4
- net COL0: track 0.00 -> 116.0 mm, vias 0 -> 6
- net COL15: track 0.00 -> 107.1 mm, vias 0 -> 5
- net COL14: track 0.00 -> 106.4 mm, vias 0 -> 4
- net COL16: track 0.00 -> 105.5 mm, vias 0 -> 4
- net COL8: track 0.00 -> 100.3 mm, vias 0 -> 5
- net COL9: track 0.00 -> 100.0 mm, vias 0 -> 5
- net COL7: track 0.00 -> 99.3 mm, vias 0 -> 5
- net COL1: track 0.00 -> 99.3 mm, vias 0 -> 5
- net COL6: track 0.00 -> 98.8 mm, vias 0 -> 5
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- added copper zone on B.Cu, net GND
- added copper zone on F.Cu, net GND
- removed copper zone on B.Cu, net GNDA
- removed copper zone on F.Cu, net GNDA

Commit message: WIP
Parts:
- removed AU: ATmega32U4-A, Package_QFP:TQFP-44_10x10mm_P0.8mm
- removed MU: QFN-44-1EP_7x7mm_P0.5mm_EP5.2x5.2mm, Package_DFN_QFN:QFN-44-1EP_7x7mm_P0.5mm_EP5.2x5.2mm
- added U1: ATmega32U4-M, Package_DFN_QFN:QFN-44-1EP_7x7mm_P0.5mm_EP5.2x5.2mm, B.Cu at (443.9, 162.9)
- SW1: value SW_Push -> Reset; footprint Button_Switch_SMD:SW_SPST_TL3342 -> cipulot_parts:Jumper-UserFriendly; moved to F.Cu
- USB1: moved to B.Cu
- moved R3 4.30 mm to (328.2, 99.0)
- moved R4 4.30 mm to (326.0, 99.0)
- moved R1 2.84 mm to (330.9, 89.6), turned to -90 degrees
- moved R2 2.68 mm to (323.3, 89.6), turned to 90 degrees
- moved SW1 2.19 mm to (470.4, 141.2), turned to 0 degrees
- moved F1 2.19 mm to (327.1, 90.5)
- moved D1 2.19 mm to (327.1, 94.2)
- turned USB1 to 0 degrees
Connections:
- R1 pad 1: GND -> Net-(R1-Pad1)
- R1 pad 2: Net-(R1-Pad2) -> GND
- R2 pad 1: Net-(R2-Pad1) -> GND
- R2 pad 2: GND -> Net-(R2-Pad2)
- SW1 pad 1: GND -> RST
- SW1 pad 2: RST -> GND
- USB1 pad 10: Net-(R2-Pad1) -> Net-(R1-Pad1)
- USB1 pad 4: Net-(R1-Pad2) -> Net-(R2-Pad2)
Routing:
- net GND: track 0.00 -> 24.6 mm, vias 0 -> 3
- net D+: track 0.00 -> 19.3 mm
- net D-: track 0.00 -> 18.2 mm
- net VBUS: track 0.00 -> 15.1 mm, vias 0 -> 3
- net Net-(R2-Pad2): track 0.00 -> 6.14 mm
- net Net-(R1-Pad1): track 0.00 -> 5.98 mm
- net VCC: track 0.00 -> 2.95 mm, vias 0 -> 1
- net COL10: track 136.9 -> 135.3 mm
- net COL13: track 125.4 -> 124.1 mm
- net COL2: track 120.7 -> 119.7 mm
- net COL11: track 121.4 -> 120.3 mm
- net COL9: track 100.0 -> 99.0 mm
- net COL8: track 100.3 -> 99.2 mm
- net COL7: track 99.3 -> 98.3 mm
- net COL6: track 98.8 -> 97.7 mm
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
Commit message: WIP
Parts:
- removed JP1: Jumper_NC_Small, Jumper:SolderJumper-2_P1.3mm_Bridged_Pad1.0x1.5mm
- removed Y1: 16MHz, cipulot_parts:Crystal_SMD_3225-4pin_3.2x2.5mm
- added C8: 1u, Capacitor_SMD:C_0603_1608Metric, B.Cu at (463.6, 161.7)
- added J1: SW Debug, Connector_PinHeader_2.54mm:PinHeader_1x04_P2.54mm_Vertical, F.Cu at (440.1, 153.1)
- added R7: 10k, Resistor_SMD:R_0805_2012Metric, B.Cu at (466.1, 147.9)
- added R8: 10k, Resistor_SMD:R_0805_2012Metric, B.Cu at (462.1, 144.1)
- added SW89: Reset, cipulot_parts:Jumper-UserFriendly, B.Cu at (439.6, 140.7)
- C1: value 0.1u -> 4.7u; footprint Capacitor_SMD:C_0805_2012Metric -> Capacitor_SMD:C_0603_1608Metric
- C2, C3: value 0.1u -> 100n; footprint Capacitor_SMD:C_0805_2012Metric -> Capacitor_SMD:C_0603_1608Metric
- C4: value 10u -> 100n; footprint Capacitor_SMD:C_0805_2012Metric -> Capacitor_SMD:C_0603_1608Metric
- C5: value 22p -> 100n; footprint Capacitor_SMD:C_0805_2012Metric -> Capacitor_SMD:C_0603_1608Metric
- C6: value 1u -> 100n; footprint Capacitor_SMD:C_0805_2012Metric -> Capacitor_SMD:C_0603_1608Metric
- C7: value 22p -> 1u; footprint Capacitor_SMD:C_0805_2012Metric -> Capacitor_SMD:C_0603_1608Metric
- R3: value 22 -> 100k
- R4: value 22 -> 10k
- SW1: value Reset -> BOOT0; moved to B.Cu
- U1: value ATmega32U4-M -> STM32F411CEUx; footprint Package_DFN_QFN:QFN-44-1EP_7x7mm_P0.5mm_EP5.2x5.2mm -> Package_DFN_QFN:QFN-48-1EP_7x7mm_P0.5mm_EP5.6x5.6mm
- moved R4 134.2 mm to (449.2, 152.3), turned to 180 degrees
- moved R3 128.2 mm to (444.8, 152.3), turned to 180 degrees
- moved C3 36.9 mm to (467.6, 159.2)
- moved U1 34.5 mm to (473.0, 144.3)
- moved C6 32.1 mm to (467.6, 156.7), turned to 180 degrees
- moved C1 27.6 mm to (467.6, 161.7), turned to 180 degrees
- moved R5 27.4 mm to (461.7, 147.1), turned to 180 degrees
- moved C4 24.4 mm to (459.6, 156.7)
- moved SW1 24.1 mm to (446.3, 141.2), turned to 180 degrees
- moved C5 16.6 mm to (463.6, 156.7), turned to 180 degrees
- moved C7 14.5 mm to (459.6, 159.2), turned to 180 degrees
- moved R6 11.9 mm to (462.1, 141.2), turned to 180 degrees
- moved C2 10.1 mm to (463.6, 159.2), turned to 180 degrees
- turned SW19 to 180 degrees
- turned SW20 to 180 degrees
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Connections:
- C1 pad 1: VCC -> Net-(C1-Pad1)
- C2 pad 1: VCC -> VDDA
- C3 pad 1: VCC -> VDDA
- C4 pad 1: VCC -> VDDA
- C5 pad 1: GND -> VDDA
- C5 pad 2: XTAL2 -> GND
- C6 pad 1: Net-(U1-Pad6) -> VDDA
- C7 pad 1: GND -> VDDA
- C7 pad 2: XTAL1 -> GND
- D1 pad 4: VCC -> +5V
- F1 pad 1: VCC -> +5V
- R1 pad 1: Net-(R1-Pad1) -> GND
- R1 pad 2: GND -> Net-(R1-Pad2)
- R2 pad 1: GND -> Net-(R2-Pad1)
- R2 pad 2: Net-(R2-Pad2) -> GND
- R3 pad 1: D+ -> Net-(R3-Pad1)
- R3 pad 2: /MCU_D+ -> VDDA
- R4 pad 1: D- -> VDDA
- R4 pad 2: /MCU_D- -> NRST
- R5 pad 1: Net-(R5-Pad1) -> PA9
- R5 pad 2: GND -> +5V
- R6 pad 1: VCC -> BOOT0
- R6 pad 2: RST -> GND
- SW1 pad 1: RST -> VDDA
- SW1 pad 2: GND -> BOOT0
- SW10 pad 1: COL9 -> COL8
- SW11 pad 1: COL10 -> COL9
- SW12 pad 1: COL11 -> COL10
- SW13 pad 1: COL12 -> COL11
- SW14 pad 1: COL13 -> COL12
- SW15 pad 1: COL14 -> COL13
- SW16 pad 1: COL15 -> COL14
- SW17 pad 1: COL16 -> COL15
- SW3 pad 1: COL2 -> COL1
- SW34 pad 1: COL16 -> COL15
- SW34 pad 2: ROW1 -> ROW2
- SW4 pad 1: COL3 -> COL2
- SW5 pad 1: COL4 -> COL3
- SW50 pad 1: COL15 -> COL14
- SW50 pad 2: ROW2 -> ROW3
- SW51 pad 1: COL16 -> COL15
- SW51 pad 2: ROW2 -> ROW3
- SW6 pad 1: COL5 -> COL4
- SW7 pad 1: COL6 -> COL5
- SW77 pad 1: COL15 -> COL14
- SW8 pad 1: COL7 -> COL6
- SW86 pad 2: ROW5 -> GND
- SW88 pad 1: COL16 -> COL15
- SW88 pad 2: ROW5 -> ROW4
- SW9 pad 1: COL8 -> COL7
- U1 pad 1: unconnected-(U1-Pad1) -> VDDA
- U1 pad 10: MOSI -> ADC
- U1 pad 11: MISO -> unconnected-(U1-Pad11)
- U1 pad 13: RST -> unconnected-(U1-Pad13)
- U1 pad 14: VCC -> unconnected-(U1-Pad14)
- U1 pad 15: GND -> unconnected-(U1-Pad15)
- U1 pad 16: XTAL2 -> unconnected-(U1-Pad16)
- U1 pad 17: XTAL1 -> unconnected-(U1-Pad17)
- U1 pad 2: VCC -> unconnected-(U1-Pad2)
- U1 pad 20: unconnected-(U1-Pad20) -> BOOT1
- U1 pad 22: unconnected-(U1-Pad22) -> Net-(C1-Pad1)
- U1 pad 24: VCC -> VDDA
- U1 pad 3: /MCU_D- -> unconnected-(U1-Pad3)
- U1 pad 30: unconnected-(U1-Pad30) -> PA9
- U1 pad 31: unconnected-(U1-Pad31) -> Net-(R3-Pad1)
- U1 pad 32: unconnected-(U1-Pad32) -> D-
- U1 pad 33: Net-(R5-Pad1) -> D+
- U1 pad 34: VCC -> SWDIO
- U1 pad 36: unconnected-(U1-Pad36) -> VDDA
- U1 pad 37: ADC -> SWCLK
- U1 pad 4: /MCU_D+ -> unconnected-(U1-Pad4)
- U1 pad 43: GND -> unconnected-(U1-Pad43)
- U1 pad 44: VCC -> BOOT0
- U1 pad 45: GND -> unconnected-(U1-Pad45)
- U1 pad 5: GND -> XTAL0
- U1 pad 6: Net-(U1-Pad6) -> XTAL1
- U1 pad 7: VCC -> NRST
- U1 pad 8: unconnected-(U1-Pad8) -> GND
- U1 pad 9: SCK -> VDDA
- USB1 pad 10: Net-(R1-Pad1) -> Net-(R2-Pad1)
- USB1 pad 4: Net-(R2-Pad2) -> Net-(R1-Pad2)
Routing:
- net ROW0: track 24.7 -> 514.0 mm, vias 16 -> 32
- net COL16: track 105.5 -> 0.00 mm, vias 4 -> 0
- net D-: track 18.2 -> 71.1 mm
- net D+: track 19.3 -> 71.9 mm
- net COL15: track 107.1 -> 142.9 mm, vias 5 -> 6
- net COL14: track 106.4 -> 139.1 mm, vias 4 -> 6
- net COL1: track 98.2 -> 129.3 mm, vias 5 -> 6
- net COL13: track 124.1 -> 96.4 mm
- net COL9: track 99.0 -> 117.8 mm
- net COL11: track 120.3 -> 135.2 mm
- net COL12: track 116.2 -> 131.0 mm
- net COL10: track 135.3 -> 149.9 mm
- net COL5: track 117.2 -> 129.0 mm
- net COL6: track 97.7 -> 107.8 mm
- net COL7: track 98.3 -> 108.1 mm
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
Commit message: Update
Parts:
- added C10: 220p, Capacitor_SMD:C_0603_1608Metric, B.Cu at (314.8, 163.3)
- added C11: 0.1u, Capacitor_SMD:C_0603_1608Metric, B.Cu at (423.2, 172.9)
- added C12: 0.1u, Capacitor_SMD:C_0603_1608Metric, B.Cu at (431.2, 180.4)
- added C13: 12p, Capacitor_SMD:C_0603_1608Metric, B.Cu at (330.8, 172.4)
- added C14: 12p, Capacitor_SMD:C_0603_1608Metric, B.Cu at (334.5, 172.4)
- added C9: 0.1u, Capacitor_SMD:C_0603_1608Metric, B.Cu at (426.9, 175.4)
- added G***: LOGO, LOGO, F.Cu at (189.4, 250.1)
- added R10: 100k, Resistor_SMD:R_0603_1608Metric, B.Cu at (416.1, 206.6)
- added R11: 100k, Resistor_SMD:R_0603_1608Metric, B.Cu at (413.9, 208.9)
- added R12: 100k, Resistor_SMD:R_0603_1608Metric, B.Cu at (416.3, 214.3)
- added R13: 100k, Resistor_SMD:R_0603_1608Metric, B.Cu at (426.3, 204.2)
- added R14: 100k, Resistor_SMD:R_0603_1608Metric, B.Cu at (430.7, 212.5)
- added R15: 100k, Resistor_SMD:R_0603_1608Metric, B.Cu at (429.3, 206.7)
- added R16: 100k, Resistor_SMD:R_0603_1608Metric, B.Cu at (430.6, 209.5)
- added R17: 100k, Resistor_SMD:R_0603_1608Metric, B.Cu at (314.8, 167.6)
- added R18: 1k, Resistor_SMD:R_0603_1608Metric, B.Cu at (313.3, 167.6)
- added R19: 100k, Resistor_SMD:R_0603_1608Metric, B.Cu at (431.9, 170.4)
- added R20: 100k, Resistor_SMD:R_0603_1608Metric, B.Cu at (431.2, 177.9)
- added R21: 100k, Resistor_SMD:R_0603_1608Metric, B.Cu at (423.2, 170.4)
- added R22: 100k, Resistor_SMD:R_0603_1608Metric, B.Cu at (418.9, 170.4)
- added R23: 100k, Resistor_SMD:R_0603_1608Metric, B.Cu at (435.6, 180.4)
- added R24: 100k, Resistor_SMD:R_0603_1608Metric, B.Cu at (439.9, 174.9)
- added R25: 100k, Resistor_SMD:R_0603_1608Metric, B.Cu at (426.9, 177.9)
- added R26: 100k, Resistor_SMD:R_0603_1608Metric, B.Cu at (427.6, 170.4)
- added R9: 100k, Resistor_SMD:R_0603_1608Metric, B.Cu at (413.4, 212.0)
- added TP1: ADC_IN, TestPoint:TestPoint_Pad_D1.0mm, B.Cu at (454.6, 191.0)
- added TP2: ADC_OUT, TestPoint:TestPoint_Pad_D1.0mm, B.Cu at (451.6, 191.0)
- added U2: 74HC4051, cipulot_parts:TSSOP16, B.Cu at (421.6, 211.3)
- added U3: OPA350, Package_SO:SOIC-8_3.9x4.9mm_P1.27mm, B.Cu at (319.4, 164.7)
- added U4: 74HC4051, cipulot_parts:TSSOP16, B.Cu at (445.2, 182.3)
- added Y1: 8MHz, Crystal:Crystal_SMD_5032-2Pin_5.0x3.2mm, B.Cu at (332.7, 168.9)
- R1: renamed from R2; footprint Resistor_SMD:R_0805_2012Metric -> Resistor_SMD:R_0603_1608Metric
- R2: renamed from R1; footprint Resistor_SMD:R_0805_2012Metric -> Resistor_SMD:R_0603_1608Metric
- R3, R4, R5, R6, R7, R8: footprint Resistor_SMD:R_0805_2012Metric -> Resistor_SMD:R_0603_1608Metric
- SW1, SW89: moved to F.Cu
- moved C1 142.0 mm to (325.7, 159.5)
- moved C3 142.0 mm to (325.7, 157.9)
- moved U1 141.9 mm to (332.1, 161.8), turned to 90 degrees
- moved C6 141.7 mm to (326.4, 168.5), turned to -90 degrees
- moved R8 137.5 mm to (325.7, 161.1), turned to 0 degrees
- moved R7 135.9 mm to (330.5, 156.4), turned to 0 degrees
- moved C7 135.0 mm to (324.9, 168.5), turned to -90 degrees
- moved R5 131.4 mm to (330.5, 154.8)
- moved R6 126.0 mm to (338.0, 162.6), turned to 0 degrees
- moved C5 125.9 mm to (338.0, 164.7), turned to 0 degrees
- moved C2 125.8 mm to (338.0, 166.3), turned to 0 degrees
- moved C8 125.8 mm to (338.0, 156.6), turned to 0 degrees
- moved R4 122.3 mm to (328.0, 168.6), turned to -90 degrees
- moved C4 121.6 mm to (338.0, 158.1), turned to 0 degrees
- moved R3 114.3 mm to (330.5, 153.3)
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Connections:
- net VDDA renamed VBAT
- R1 pad 1: Net-(R2-Pad1) -> GND
- R1 pad 2: GND -> Net-(R1-Pad2)
- R2 pad 1: GND -> Net-(R2-Pad1)
- R2 pad 2: Net-(R1-Pad2) -> GND
- SW10 pad 2: ROW0 -> SWCLK
- SW11 pad 2: ROW0 -> SWCLK
- SW12 pad 2: ROW0 -> SWCLK
- SW13 pad 2: ROW0 -> SWCLK
- SW14 pad 2: ROW0 -> SWCLK
- SW15 pad 2: ROW0 -> SWCLK
- SW16 pad 2: ROW0 -> SWCLK
- SW17 pad 2: ROW0 -> SWCLK
- SW2 pad 2: ROW0 -> SWCLK
- SW3 pad 2: ROW0 -> SWCLK
- SW4 pad 2: ROW0 -> SWCLK
- SW5 pad 2: ROW0 -> SWCLK
- SW6 pad 2: ROW0 -> SWCLK
- SW7 pad 2: ROW0 -> SWCLK
- SW8 pad 2: ROW0 -> SWCLK
- SW9 pad 2: ROW0 -> SWCLK
- U1 pad 10: ADC -> unconnected-(U1-Pad10)
- U1 pad 12: unconnected-(U1-Pad12) -> POWER_PIN
- U1 pad 14: unconnected-(U1-Pad14) -> ADC
- U1 pad 38: unconnected-(U1-Pad38) -> ROW1
- U1 pad 39: unconnected-(U1-Pad39) -> ROW2
- U1 pad 40: unconnected-(U1-Pad40) -> ROW3
- U1 pad 41: unconnected-(U1-Pad41) -> ROW4
- U1 pad 42: unconnected-(U1-Pad42) -> ROW5
Routing:
- net SWCLK: track 0.00 -> 514.0 mm, vias 0 -> 32
- net ROW0: track 514.0 -> 0.00 mm, vias 32 -> 0
- net VBAT: track 0.00 -> 53.0 mm, vias 0 -> 4
- net GND: track 25.4 -> 43.8 mm, vias 4 -> 19
- net ADC: track 0.00 -> 17.3 mm
- net D-: track 71.1 -> 81.3 mm
- net D+: track 71.9 -> 82.1 mm
- net POWER_PIN: track 0.00 -> 8.04 mm
- net XTAL0: track 0.00 -> 7.03 mm
- net XTAL1: track 0.00 -> 7.00 mm
- net NRST: track 0.00 -> 6.87 mm
- net Net-(R3-Pad1): track 0.00 -> 5.46 mm
- net Net-(R17-Pad2): track 0.00 -> 4.65 mm
- net PA9: track 0.00 -> 3.73 mm
- net Net-(C1-Pad1): track 0.00 -> 2.45 mm
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