File: PCB/EC87.kicad_sch (KiCad schematic)
At the start: 21 parts, among them J1 AVR-ISP-6-Connector, SW1 SW_Push, U1 ATmega32U4-A, Y1 16MHz

Commit message: WIP
Parts:
- renumbered JP2 to JP1

Commit message: WIP
Parts:
- removed J1: AVR-ISP-6-Connector, cipulot_parts:Reset_Pretty, symbol cipulot_parts:AVR-ISP-6-Connector

Commit message: WIP
Parts:
- removed SW1: SW_Push, Button_Switch_SMD:SW_SPST_TL3342, symbol Switch:SW_Push
- removed U1: ATmega32U4-A, Package_QFP:TQFP-44_10x10mm_P0.8mm, symbol MCU_Microchip_ATmega:ATmega32U4-A
- added SW1: Reset, cipulot_parts:Jumper-UserFriendly, symbol Jumper:Jumper_2_Open
- added U1: ATmega32U4-M, Package_DFN_QFN:QFN-44-1EP_7x7mm_P0.5mm_EP5.2x5.2mm, symbol MCU_Microchip_ATmega:ATmega32U4-M
- renumbered R2 to R1, R1 to R2
Connections:
- net ADC: now also U1.37 (PF6)
- net GND: now also SW1.2 (B), U1.15 (GND), U1.23 (GND), U1.35 (GND), U1.43 (GND), U1.45 (GND), U1.5 (UGND)
- net MCU_D+: now also U1.4 (D+)
- net MCU_D-: now also U1.3 (D-)
- net MISO: now also U1.11 (PB3)
- net MOSI: now also U1.10 (PB2)
- net RST: now also SW1.1 (A), U1.13 (~{RESET})
- net SCK: now also U1.9 (PB1)
- net VCC: now also U1.14 (VCC), U1.2 (UVCC), U1.24 (AVCC), U1.34 (VCC), U1.44 (AVCC), U1.7 (VBUS)
- net XTAL1: now also U1.17 (XTAL1)
- net XTAL2: now also U1.16 (XTAL2)
- net at R5.1: now also U1.33 (~{HWB}/PE2)
- net at C6.1: now also U1.6 (UCAP)

Commit message: WIP
Parts:
- removed JP1: Jumper_NC_Small, Jumper:SolderJumper-2_P1.3mm_Bridged_Pad1.0x1.5mm, symbol Device:Jumper_NC_Small
- removed R4: 22, Resistor_SMD:R_0805_2012Metric, symbol Device:R
- removed U1: ATmega32U4-M, Package_DFN_QFN:QFN-44-1EP_7x7mm_P0.5mm_EP5.2x5.2mm, symbol MCU_Microchip_ATmega:ATmega32U4-M
- removed Y1: 16MHz, cipulot_parts:Crystal_SMD_3225-4pin_3.2x2.5mm, symbol Device:Crystal_GND24
- added C8: 1u, Capacitor_SMD:C_0603_1608Metric, symbol Device:C
- added J1: SW Debug, Connector_PinHeader_2.54mm:PinHeader_1x04_P2.54mm_Vertical, symbol Connector_Generic:Conn_01x04
- added R6, R7, R8: 10k, Resistor_SMD:R_0805_2012Metric, symbol Device:R
- added SW1: BOOT0, cipulot_parts:Jumper-UserFriendly, symbol Jumper:Jumper_2_Open
- added U1: STM32F411CEUx, Package_DFN_QFN:QFN-48-1EP_7x7mm_P0.5mm_EP5.6x5.6mm, symbol MCU_ST_STM32F4:STM32F411CEUx
- C1: value 0.1u -> 4.7u; footprint Capacitor_SMD:C_0805_2012Metric -> Capacitor_SMD:C_0603_1608Metric
- C2, C3: value 0.1u -> 100n; footprint Capacitor_SMD:C_0805_2012Metric -> Capacitor_SMD:C_0603_1608Metric
- C4: value 10u -> 100n; footprint Capacitor_SMD:C_0805_2012Metric -> Capacitor_SMD:C_0603_1608Metric
- C5: value 22p -> 100n; footprint Capacitor_SMD:C_0805_2012Metric -> Capacitor_SMD:C_0603_1608Metric
- C6: value 1u -> 100n; footprint Capacitor_SMD:C_0805_2012Metric -> Capacitor_SMD:C_0603_1608Metric
- C7: value 22p -> 1u; footprint Capacitor_SMD:C_0805_2012Metric -> Capacitor_SMD:C_0603_1608Metric
- R3: value 22 -> 100k
- renumbered R2 to R1, R1 to R2, R6 to R4, SW1 to SW89
Connections:
- net MCU_D+ is gone; now on net +3V3: R3.2
- net XTAL2 is gone; now on net GND: C5.2
- net +5V: now also D1.4 (VCC), F1.1, R5.2
- net ADC: now also U1.10 (PA0)
- net D+: now also U1.33 (PA12); no longer R3.1
- net D-: now also U1.32 (PA11)
- net GND: now also C7.2, C8.2, J1.4 (Pin_4), R6.2, R7.1, R8.1, U1.23 (VSS), U1.35 (VSS), U1.47 (VSS), U1.49 (VSS), U1.8 (VSSA); no longer C5.1, C7.1, R5.2
- net VCC: no longer C1.1, C2.1, C3.1, C4.1, D1.4 (VCC), F1.1, R4.1
- net XTAL1: now also U1.6 (PH1); no longer C7.2
- net PA9: now reaches R5.1
- net PA9: now also R7.2, U1.30 (PA9)
- net +3V3: now reaches C6.1
- net +3V3: now also C2.1, C3.1, C4.1, C5.1, C7.1, R4.1, C8.1, J1.1 (Pin_1), SW1.1 (A), U1.1 (VBAT), U1.24 (VDD), U1.36 (VDD), U1.48 (VDD), U1.9 (VDDA)
- net RST renamed NRST
- net NRST: now also U1.7 (NRST)
- new net: C1.1, U1.22 (VCAP1)
- new net: R3.1, U1.31 (PA10)
- new net BOOT0: R6.1, SW1.2 (B), U1.44 (BOOT0)
- new net BOOT1: R8.2, U1.20 (PB2)
- new net SWCLK: J1.3 (Pin_3), U1.37 (PA14)
- new net SWDIO: J1.2 (Pin_2), U1.34 (PA13)
- new net XTAL0: U1.5 (PH0)
- no-connect marks 3 -> 2
Other:
- note added: "BOOT0 Switch"
- note added: "Decoupling Capacitors"
- note added: "Reset Switch"
- note added: "SW Debug Breakout"
- note added: "Weird Stuff FIx"
- moved on the sheet: F1, R1, R2, R4, SW89, USB1

Commit message: Update
Parts:
- added C13, C14: 12p, Capacitor_SMD:C_0603_1608Metric, symbol Device:C
- added Y1: 8MHz, Crystal:Crystal_SMD_5032-2Pin_5.0x3.2mm, symbol Device:Crystal
- R1, R2, R3, R4, R5, R6, R7, R8: footprint Resistor_SMD:R_0805_2012Metric -> Resistor_SMD:R_0603_1608Metric
Connections:
- net ADC: now also U1.14 (PA4); no longer U1.10 (PA0)
- net GND: now also C13.2, C14.2
- net XTAL0: now also C14.1, Y1.2
- net XTAL1: now also C13.1, Y1.1
- net POWER_PIN: now reaches U1.12 (PA2)
- net ROW1: now reaches U1.38 (PA15)
- net ROW2: now reaches U1.39 (PB3)
- net ROW3: now reaches U1.40 (PB4)
- net ROW4: now reaches U1.41 (PB5)
- net ROW5: now reaches U1.42 (PB6)
- net SWCLK renamed ROW0
- no-connect marks 2 -> 11

Commit message: Update
Parts:
- added C15, C16: 1u, Capacitor_SMD:C_0603_1608Metric, symbol Device:C
- added U5: XC6206PxxxMR, Package_TO_SOT_SMD:SOT-23, symbol Regulator_Linear:XC6206PxxxMR
Connections:
- net POWER_PIN is gone; now on net ADC: U1.12 (PA2)
- net +3V3: now also C16.1, U5.2 (VO)
- net +5V: now also C15.1, U5.3 (VI)
- net ADC: no longer U1.14 (PA4)
- net AMUX_SEL_0: now also U1.17 (PA7)
- net AMUX_SEL_1: now also U1.16 (PA6)
- net AMUX_SEL_2: now also U1.15 (PA5)
- net APLEX_EN_PIN_0: now also U1.18 (PB0)
- net APLEX_EN_PIN_1: now also U1.43 (PB7)
- net GND: now also C15.2, C16.2, U5.1 (GND)
- net ROW0: now also U1.40 (PB4); no longer J1.3 (Pin_3), U1.37 (PA14)
- net ROW1: now also J1.3 (Pin_3), U1.37 (PA14); no longer U1.38 (PA15)
- net ROW2: now also U1.38 (PA15); no longer U1.39 (PB3)
- net ROW3: now also U1.39 (PB3); no longer U1.40 (PB4)
- no-connect marks 11 -> 10
Other:
- note added: "Voltage Regulator"
