File: PCB/EC87.kicad_sch (KiCad schematic)
At the start: 27 parts, among them J1 SW Debug, SW1 BOOT0, SW89 Reset, U1 STM32F411CEUx, U5 XC6206PxxxMR, Y1 8MHz

Commit message: Update of schematic infos and backplate
Other:
- company: (none) -> Cipulot's PCB Design 
- title: (none) -> EC87
Changed lines of the file:
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@@
 (kicad_sch (version 20211123) (generator eeschema)
   (paper "A4")
+  (title_block
+    (title "EC87")
+    (date "2022-03-30")
+    (rev "1")
+    (company "Cipulot's PCB Design ")
+    (comment 2 "Cipulot")
+  )
   (junction (at 92.71 177.8) (diameter 0) (color 0 0 0 0)
   )
