File: PCB/backplate.kicad_pcb (KiCad board)
At the start: 2 copper layers, 354 x 121 mm, 40 parts

Commit message: Update of backplate
Parts:
- removed the ? at (351.4, 155.6)
- removed the ? at (65.5, 136.6)
- removed the ? at (367.1, 136.6)
- removed the ? at (115.3, 117.5)
- removed the ? at (42.3, 155.6)
- removed the ? at (325.5, 193.6)
- removed the ? at (234.1, 174.6)
- removed the ? at (243.6, 93.8)
- removed the ? at (267.3, 117.5)
- removed the ? at (348.1, 117.5)
- removed the ? at (367.1, 193.6)
- removed the ? at (96.3, 93.8)
- removed the ? at (253.1, 193.6)
- removed the ? at (91.6, 155.6)
- removed the ? at (148.6, 193.6)
- removed the ? at (300.6, 193.6)
- removed the ? at (367.1, 93.7)
- removed the ? at (276.8, 136.6)
- removed the ? at (139.1, 174.6)
- removed the ? at (376.6, 174.6)
- removed the ? at (191.3, 117.5)
- removed the ? at (181.8, 93.8)
- removed the ? at (143.8, 136.6)
- removed the ? at (283.7, 161.9)
- removed the ? at (67.8, 93.8)
- removed the ? at (63.1, 193.6)
- removed the ? at (58.3, 117.5)
- removed the ? at (186.6, 155.6)
- removed the ? at (286.3, 93.8)
- removed the ? at (110.6, 193.6)
- removed the ? at (191.3, 193.6)
- moved G*** 32.6 mm to (281.4, 143.7)

Commit message: Update backplate silkscreen
Parts:
- added ?: , , F.Cu at (186.6, 155.6)
- added ?: , kbd:M2_Hole_TH, F.Cu at (181.8, 93.8)
- added ?: , , F.Cu at (42.3, 155.6)
- added ?: , kbd:M2_Hole_TH, F.Cu at (148.6, 193.6)
- added ?: , , F.Cu at (376.6, 174.6)
- added ?: , kbd:M2_Hole_TH, F.Cu at (139.1, 174.6)
- added ?: , kbd:M2_Hole_TH, F.Cu at (65.5, 136.6)
- added ?: , , F.Cu at (67.8, 93.8)
- added ?: , , F.Cu at (276.8, 136.6)
- added ?: , kbd:M2_Hole_TH, F.Cu at (63.1, 193.6)
- added ?: , , F.Cu at (234.1, 174.6)
- added ?: , , F.Cu at (91.6, 155.6)
- added ?: , kbd:M2_Hole_TH, F.Cu at (191.3, 193.6)
- added ?: , kbd:M2_Hole_TH, F.Cu at (58.3, 117.5)
- added ?: , , F.Cu at (348.1, 117.5)
- added ?: , , F.Cu at (325.5, 193.6)
- added ?: , , F.Cu at (300.6, 193.6)
- added ?: , , F.Cu at (267.3, 117.5)
- added ?: , , F.Cu at (115.3, 117.5)
- added ?: , , F.Cu at (367.1, 193.6)
- added ?: , , F.Cu at (286.3, 93.8)
- added ?: , , F.Cu at (367.1, 93.7)
- added ?: , , F.Cu at (283.7, 161.9)
- added ?: , , F.Cu at (351.4, 155.6)
- added ?: , , F.Cu at (253.1, 193.6)
- added ?: , , F.Cu at (191.3, 117.5)
- added ?: , , F.Cu at (96.3, 93.8)
- added ?: , kbd:M2_Hole_TH, F.Cu at (110.6, 193.6)
- added ?: , , F.Cu at (367.1, 136.6)
- added ?: , , F.Cu at (143.8, 136.6)
- added ?: , kbd:M2_Hole_TH, F.Cu at (243.6, 93.8)
- added G***: LOGO, LOGO, F.Cu at (214.4, 123.0)
- added G***: LOGO, LOGO, B.Cu at (219.7, 155.6)
- moved G*** 32.3 mm to (313.5, 140.1)

Commit message: Update of schematic infos and backplate
Parts:
- removed the G*** at (214.4, 123.0)
