File: PCB/matrix.kicad_sch (KiCad schematic)
At the start: 87 parts, among them SW10 EC_SW, SW11 EC_SW, SW12 EC_SW, SW13 EC_SW, SW14 EC_SW, SW15 EC_SW, SW16 EC_SW, SW17 EC_SW, SW18 EC_SW, SW19 EC_SW, SW2 EC_SW, SW20 EC_SW, SW21 EC_SW, SW22 EC_SW, SW23 EC_SW, SW24 EC_SW, SW25 EC_SW, SW26 EC_SW, SW27 EC_SW, SW28 EC_SW, SW29 EC_SW, SW3 EC_SW, SW30 EC_SW, SW31 EC_SW, SW32 EC_SW, SW33 EC_SW, SW34 EC_SW, SW35 EC_SW, SW36 EC_SW, SW37 EC_SW, SW38 EC_SW, SW39 EC_SW, SW4 EC_SW, SW40 EC_SW, SW41 EC_SW, SW42 EC_SW, SW43 EC_SW, SW44 EC_SW, SW45 EC_SW, SW46 EC_SW, SW47 EC_SW, SW48 EC_SW, SW49 EC_SW, SW5 EC_SW, SW50 EC_SW, SW51 EC_SW, SW52 EC_SW, SW53 EC_SW, SW54 EC_SW, SW55 EC_SW, SW56 EC_SW, SW57 EC_SW, SW58 EC_SW, SW59 EC_SW, SW6 EC_SW, SW60 EC_SW, SW61 EC_SW, SW62 EC_SW, SW63 EC_SW, SW64 EC_SW, SW65 EC_SW, SW66 EC_SW, SW67 EC_SW, SW68 EC_SW, SW69 EC_SW, SW7 EC_SW, SW70 EC_SW, SW71 EC_SW, SW72 EC_SW, SW73 EC_SW, SW74 EC_SW, SW75 EC_SW, SW76 EC_SW, SW77 EC_SW, SW78 EC_SW, SW79 EC_SW, SW8 EC_SW, SW80 EC_SW, SW81 EC_SW, SW82 EC_SW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

Commit message: WIP
Parts:
- added SW? (x4): EC_SW, cipulot_parts:ecs_pad, symbol cipulot_parts:EC_SW
Connections:
- net COL11: now also SW?.1
- net COL3: now also SW?.1
- net COL9: now also SW?.1
- net GNDA: now also SW?.3 (SG), SW?.3 (SG), SW?.3 (SG), SW?.3 (SG)
- net ROW1: now also SW?.2
- net ROW4: now also SW?.2
- net ROW5: now also SW?.2, SW?.2
Changed lines of the file:
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@@
   (junction (at 250.19 96.52) (diameter 0) (color 0 0 0 0)
   )
+  (junction (at 99.06 153.67) (diameter 0) (color 0 0 0 0)
+  )
   (junction (at 96.52 160.02) (diameter 0) (color 0 0 0 0)
   )
@@
   (junction (at 78.74 118.11) (diameter 0) (color 0 0 0 0)
   )
+  (junction (at 114.3 173.99) (diameter 0) (color 0 0 0 0)
+  )
   (junction (at 152.4 125.73) (diameter 0) (color 0 0 0 0)
   )
@@
   (junction (at 78.74 173.99) (diameter 0) (color 0 0 0 0)
   )
+  (junction (at 303.53 116.84) (diameter 0) (color 0 0 0 0)
+  )
   (junction (at 259.08 125.73) (diameter 0) (color 0 0 0 0)
   )
@@
   (junction (at 88.9 144.78) (diameter 0) (color 0 0 0 0)
   )
+  (junction (at 241.3 153.67) (diameter 0) (color 0 0 0 0)
+  )
   (junction (at 45.72 111.76) (diameter 0) (color 0 0 0 0)
   )
@@
   (junction (at 223.52 111.76) (diameter 0) (color 0 0 0 0)
   )
+  (junction (at 106.68 172.72) (diameter 0) (color 0 0 0 0)
+  )
   (junction (at 341.63 132.08) (diameter 0) (color 0 0 0 0)
   )
+  (junction (at 220.98 173.99) (diameter 0) (color 0 0 0 0)
+  )
   (junction (at 326.39 91.44) (diameter 0) (color 0 0 0 0)
   )
@@
   (junction (at 203.2 118.11) (diameter 0) (color 0 0 0 0)
   )
+  (junction (at 256.54 160.02) (diameter 0) (color 0 0 0 0)
+  )
   (junction (at 81.28 139.7) (diameter 0) (color 0 0 0 0)
   )
@@
   (junction (at 361.95 91.44) (diameter 0) (color 0 0 0 0)
   )
+  (junction (at 248.92 158.75) (diameter 0) (color 0 0 0 0)
+  )
   (junction (at 213.36 99.06) (diameter 0) (color 0 0 0 0)
   )
@@
   (junction (at 231.14 158.75) (diameter 0) (color 0 0 0 0)
   )
+  (junction (at 311.15 118.11) (diameter 0) (color 0 0 0 0)
+  )
   (junction (at 341.63 99.06) (diameter 0) (color 0 0 0 0)
   )
@@
   (junction (at 351.79 116.84) (diameter 0) (color 0 0 0 0)
   )
+  (junction (at 205.74 153.67) (diameter 0) (color 0 0 0 0)
+  )
   (junction (at 60.96 132.08) (diameter 0) (color 0 0 0 0)
   )
@@
   (junction (at 213.36 116.84) (diameter 0) (color 0 0 0 0)
   )
+  (junction (at 213.36 172.72) (diameter 0) (color 0 0 0 0)
+  )
   (junction (at 276.86 153.67) (diameter 0) (color 0 0 0 0)
   )
@@
     (stroke (width 0) (type default) (color 0 0 0 0))
   )
+  (wire (pts (xy 220.98 173.99) (xy 238.76 173.99))
+    (stroke (width 0) (type default) (color 0 0 0 0))
+  )
   (wire (pts (xy 359.41 125.73) (xy 359.41 132.08))
     (stroke (width 0) (type default) (color 0 0 0 0))
@@
     (stroke (width 0) (type default) (color 0 0 0 0))
   )
+  (wire (pts (xy 241.3 153.67) (xy 241.3 167.64))
+    (stroke (width 0) (type default) (color 0 0 0 0))
+  )
   (wire (pts (xy 278.13 102.87) (xy 278.13 91.44))
     (stroke (width 0) (type default) (color 0 0 0 0))
@@
     (stroke (width 0) (type default) (color 0 0 0 0))
   )
+  (wire (pts (xy 311.15 118.11) (xy 341.63 118.11))
+    (stroke (width 0) (type default) (color 0 0 0 0))
+  )
   (wire (pts (xy 60.96 167.64) (xy 60.96 173.99))
     (stroke (width 0) (type default) (color 0 0 0 0))
@@
     (stroke (width 0) (type default) (color 0 0 0 0))
   )
+  (wire (pts (xy 248.92 158.75) (xy 284.48 158.75))
+    (stroke (width 0) (type default) (color 0 0 0 0))
+  )
   (wire (pts (xy 292.1 111.76) (xy 292.1 118.11))
     (stroke (width 0) (type default) (color 0 0 0 0))
@@
     (stroke (width 0) (type default) (color 0 0 0 0))
   )
+  (wire (pts (xy 256.54 153.67) (xy 256.54 160.02))
+    (stroke (width 0) (type default) (color 0 0 0 0))
+  )
   (wire (pts (xy 275.59 99.06) (xy 293.37 99.06))
     (stroke (width 0) (type default) (color 0 0 0 0))
@@
     (stroke (width 0) (type default) (color 0 0 0 0))
   )
-  (wire (pts (xy 161.29 173.99) (xy 238.76 173.99))
+  (wire (pts (xy 161.29 173.99) (xy 220.98 173.99))
     (stroke (width 0) (type default) (color 0 0 0 0))
   )
@@
     (stroke (width 0) (type default) (color 0 0 0 0))
   )
+  (wire (pts (xy 99.06 153.67) (xy 99.06 167.64))
+    (stroke (width 0) (type default) (color 0 0 0 0))
+  )
   (wire (pts (xy 215.9 101.6) (xy 215.9 91.44))
     (stroke (width 0) (type default) (color 0 0 0 0))
@@
     (stroke (width 0) (type default) (color 0 0 0 0))
   )
-  (wire (pts (xy 284.48 116.84) (xy 334.01 116.84))
+  (wire (pts (xy 284.48 116.84) (xy 303.53 116.84))
     (stroke (width 0) (type default) (color 0 0 0 0))
   )
@@
     (stroke (width 0) (type default) (color 0 0 0 0))
   )
-  (wire (pts (xy 231.14 158.75) (xy 284.48 158.75))
+  (wire (pts (xy 231.14 158.75) (xy 248.92 158.75))
+    (stroke (width 0) (type default) (color 0 0 0 0))
+  )
+  (wire (pts (xy 114.3 173.99) (xy 161.29 173.99))
     (stroke (width 0) (type default) (color 0 0 0 0))
   )
@@
     (stroke (width 0) (type default) (color 0 0 0 0))
   )
+  (wire (pts (xy 106.68 172.72) (xy 153.67 172.72))
+    (stroke (width 0) (type default) (color 0 0 0 0))
+  )
   (wire (pts (xy 96.52 99.06) (xy 114.3 99.06))
     (stroke (width 0) (type default) (color 0 0 0 0))
@@
     (stroke (width 0) (type default) (color 0 0 0 0))
   )
+  (wire (pts (xy 114.3 167.64) (xy 114.3 173.99))
+    (stroke (width 0) (type default) (color 0 0 0 0))
+  )
   (wire (pts (xy 60.96 118.11) (xy 78.74 118.11))
     (stroke (width 0) (type default) (color 0 0 0 0))
   )
+  (wire (pts (xy 303.53 116.84) (xy 334.01 116.84))
+    (stroke (width 0) (type default) (color 0 0 0 0))
+  )
   (wire (pts (xy 341.63 167.64) (xy 341.63 173.99))
     (stroke (width 0) (type default) (color 0 0 0 0))
@@
     (stroke (width 0) (type default) (color 0 0 0 0))
   )
-  (wire (pts (xy 238.76 160.02) (xy 292.1 160.02))
+  (wire (pts (xy 238.76 160.02) (xy 256.54 160.02))
     (stroke (width 0) (type default) (color 0 0 0 0))
   )
@@
     (stroke (width 0) (type default) (color 0 0 0 0))
   )
-  (wire (pts (xy 153.67 172.72) (xy 231.14 172.72))
+  (wire (pts (xy 220.98 167.64) (xy 220.98 173.99))
+    (stroke (width 0) (type default) (color 0 0 0 0))
+  )
+  (wire (pts (xy 153.67 172.72) (xy 213.36 172.72))
+    (stroke (width 0) (type default) (color 0 0 0 0))
+  )
+  (wire (pts (xy 205.74 153.67) (xy 205.74 167.64))
     (stroke (width 0) (type default) (color 0 0 0 0))
   )
@@
     (stroke (width 0) (type default) (color 0 0 0 0))
   )
-  (wire (pts (xy 292.1 118.11) (xy 341.63 118.11))
+  (wire (pts (xy 292.1 118.11) (xy 311.15 118.11))
     (stroke (width 0) (type default) (color 0 0 0 0))
   )
@@
     (stroke (width 0) (type default) (color 0 0 0 0))
   )
+  (wire (pts (xy 311.15 111.76) (xy 311.15 118.11))
+    (stroke (width 0) (type default) (color 0 0 0 0))
+  )
   (wire (pts (xy 185.42 132.08) (xy 203.2 132.08))
     (stroke (width 0) (type default) (color 0 0 0 0))
@@
     (stroke (width 0) (type default) (color 0 0 0 0))
   )
-  (wire (pts (xy 241.3 139.7) (xy 241.3 167.64))
+  (wire (pts (xy 241.3 139.7) (xy 241.3 153.67))
     (stroke (width 0) (type default) (color 0 0 0 0))
   )
@@
     (stroke (width 0) (type default) (color 0 0 0 0))
   )
-  (wire (pts (xy 96.52 173.99) (xy 161.29 173.99))
+  (wire (pts (xy 256.54 160.02) (xy 292.1 160.02))
+    (stroke (width 0) (type default) (color 0 0 0 0))
+  )
+  (wire (pts (xy 96.52 173.99) (xy 114.3 173.99))
     (stroke (width 0) (type default) (color 0 0 0 0))
   )
@@
     (stroke (width 0) (type default) (color 0 0 0 0))
   )
+  (wire (pts (xy 213.36 172.72) (xy 231.14 172.72))
+    (stroke (width 0) (type default) (color 0 0 0 0))
+  )
   (wire (pts (xy 284.48 130.81) (xy 334.01 130.81))
     (stroke (width 0) (type default) (color 0 0 0 0))
@@
     (stroke (width 0) (type default) (color 0 0 0 0))
   )
-  (wire (pts (xy 88.9 172.72) (xy 153.67 172.72))
+  (wire (pts (xy 88.9 172.72) (xy 106.68 172.72))
     (stroke (width 0) (type default) (color 0 0 0 0))
   )
@@
     (pin "3")
   )
+  (symbol (lib_id "cipulot_parts:EC_SW") (at 303.53 111.76 0) (unit 1)
+    (in_bom yes) (on_board yes) (fields_autoplaced)
+    (property "Reference" "SW?" (id 0) (at 303.53 105.6345 0))
+    (property "Value" "EC_SW" (id 1) (at 303.53 108.4096 0))
+    (property "Footprint" "cipulot_parts:ecs_pad" (id 2) (at 303.53 111.76 0)
+      (effects (font (size 1.27 1.27)) hide)
+    )
+    (property "Datasheet" "" (id 3) (at 303.53 111.76 0))
+    (pin "1")
+    (pin "2")
+    (pin "3")
+  )
   (symbol (lib_id "cipulot_parts:EC_SW") (at 213.36 153.67 0) (unit 1)
     (in_bom yes) (on_board yes) (fields_autoplaced)
@@
     (pin "3")
   )
+  (symbol (lib_id "cipulot_parts:EC_SW") (at 213.36 167.64 0) (unit 1)
+    (in_bom yes) (on_board yes) (fields_autoplaced)
+    (property "Reference" "SW?" (id 0) (at 213.36 161.5145 0))
+    (property "Value" "EC_SW" (id 1) (at 213.36 164.2896 0))
+    (property "Footprint" "cipulot_parts:ecs_pad" (id 2) (at 213.36 167.64 0)
+      (effects (font (size 1.27 1.27)) hide)
+    )
+    (property "Datasheet" "" (id 3) (at 213.36 167.64 0))
+    (pin "1")
+    (pin "2")
+    (pin "3")
+  )
+  (symbol (lib_id "cipulot_parts:EC_SW") (at 106.68 167.64 0) (unit 1)
+    (in_bom yes) (on_board yes) (fields_autoplaced)
+    (property "Reference" "SW?" (id 0) (at 106.68 161.5145 0))
+    (property "Value" "EC_SW" (id 1) (at 106.68 164.2896 0))
+    (property "Footprint" "cipulot_parts:ecs_pad" (id 2) (at 106.68 167.64 0)
+      (effects (font (size 1.27 1.27)) hide)
+    )
+    (property "Datasheet" "" (id 3) (at 106.68 167.64 0))
+    (pin "1")
+    (pin "2")
+    (pin "3")
+  )
   (symbol (lib_id "cipulot_parts:EC_SW") (at 248.92 111.76 0) (unit 1)
     (in_bom yes) (on_board yes) (fields_autoplaced)
@@
     (pin "1")
     (pin "2")
+    (pin "3")
+  )
+  (symbol (lib_id "cipulot_parts:EC_SW") (at 248.92 153.67 0) (unit 1)
+    (in_bom yes) (on_board yes) (fields_autoplaced)
+    (property "Reference" "SW?" (id 0) (at 248.92 147.5445 0))
+    (property "Value" "EC_SW" (id 1) (at 248.92 150.3196 0))
+    (property "Footprint" "cipulot_parts:ecs_pad" (id 2) (at 248.92 153.67 0)
+      (effects (font (size 1.27 1.27)) hide)
+    )
+    (property "Datasheet" "" (id 3) (at 248.92 153.67 0))
+    (pin "1")
+    (pin "2")

Commit message: WIP
Parts:
- gave numbers to parts that had none: 4
- renumbered SW32 to SW33, SW33 to SW34, SW34 to SW35, SW35 to SW36, SW36 to SW37, SW37 to SW38, SW38 to SW39, SW39 to SW40, SW40 to SW41, SW41 to SW42, SW42 to SW43, SW43 to SW44, SW44 to SW45, SW45 to SW46, SW46 to SW47, SW47 to SW48, SW48 to SW49, SW49 to SW50, SW50 to SW51, SW51 to SW52, SW52 to SW53, SW53 to SW54, SW54 to SW55, SW55 to SW56, SW56 to SW57, SW57 to SW58, SW58 to SW59, SW59 to SW60, SW60 to SW61, SW61 to SW62, SW62 to SW63, SW63 to SW64, SW64 to SW65, SW65 to SW66, SW66 to SW67, SW67 to SW68, SW68 to SW69, SW69 to SW70, SW70 to SW71, SW71 to SW72, SW72 to SW73, SW73 to SW74, SW74 to SW75, SW75 to SW76, SW76 to SW78, SW77 to SW79, SW78 to SW80, SW79 to SW81, SW80 to SW82, SW81 to SW84, SW82 to SW86, SW83 to SW87, SW84 to SW88, SW85 to SW89, SW86 to SW90, SW87 to SW91, SW88 to SW92

Commit message: WIP
Parts:
- removed SW32, SW77, SW83, SW85: EC_SW, cipulot_parts:ecs_pad, symbol cipulot_parts:EC_SW
- renumbered SW33 to SW32, SW34 to SW33, SW35 to SW34, SW36 to SW35, SW37 to SW36, SW38 to SW37, SW39 to SW38, SW40 to SW39, SW41 to SW40, SW42 to SW41, SW43 to SW42, SW44 to SW43, SW45 to SW44, SW46 to SW45, SW47 to SW46, SW48 to SW47, SW49 to SW48, SW50 to SW49, SW51 to SW50, SW52 to SW51, SW53 to SW52, SW54 to SW53, SW55 to SW54, SW56 to SW55, SW57 to SW56, SW58 to SW57, SW59 to SW58, SW60 to SW59, SW61 to SW60, SW62 to SW61, SW63 to SW62, SW64 to SW63, SW65 to SW64, SW66 to SW65, SW67 to SW66, SW68 to SW67, SW69 to SW68, SW70 to SW69, SW71 to SW70, SW72 to SW71, SW73 to SW72, SW74 to SW73, SW75 to SW74, SW76 to SW75, SW78 to SW76, SW79 to SW77, SW80 to SW78, SW81 to SW79, SW82 to SW80, SW84 to SW81, SW86 to SW82, SW87 to SW83, SW88 to SW84, SW89 to SW85, SW90 to SW86, SW91 to SW87, SW92 to SW88
Connections:
- net GNDA renamed GND

Commit message: WIP
Connections:
- net COL16 is gone; now on net COL15: SW17.1, SW34.1, SW51.1, SW88.1
- net COL1: now also SW3.1
- net COL10: now also SW12.1; no longer SW11.1
- net COL11: now also SW13.1; no longer SW12.1
- net COL12: now also SW14.1; no longer SW13.1
- net COL13: now also SW15.1; no longer SW14.1
- net COL14: now also SW16.1, SW50.1, SW77.1; no longer SW15.1
- net COL15: no longer SW16.1, SW50.1, SW77.1
- net COL2: now also SW4.1; no longer SW3.1
- net COL3: now also SW5.1; no longer SW4.1
- net COL4: now also SW6.1; no longer SW5.1
- net COL5: now also SW7.1; no longer SW6.1
- net COL6: now also SW8.1; no longer SW7.1
- net COL7: now also SW9.1; no longer SW8.1
- net COL8: now also SW10.1; no longer SW9.1
- net COL9: now also SW11.1; no longer SW10.1
- net GND: now also SW86.2
- net ROW1: no longer SW34.2
- net ROW2: now also SW34.2; no longer SW50.2, SW51.2
- net ROW3: now also SW50.2, SW51.2
- net ROW4: now also SW88.2
- net ROW5: no longer SW86.2, SW88.2

Commit message: Update
Connections:
- net GND: no longer SW86.2
- net ROW4: now also SW66.2
- net ROW5: now also SW86.2
Changed lines of the file:
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@@
   (junction (at 213.36 144.78) (diameter 0) (color 0 0 0 0)
   )
+  (junction (at 323.85 173.99) (diameter 0) (color 0 0 0 0)
+  )
   (junction (at 334.01 96.52) (diameter 0) (color 0 0 0 0)
   )
@@
   (junction (at 284.48 172.72) (diameter 0) (color 0 0 0 0)
   )
+  (junction (at 78.74 160.02) (diameter 0) (color 0 0 0 0)
+  )
   (junction (at 88.9 144.78) (diameter 0) (color 0 0 0 0)
   )
@@
   (junction (at 81.28 111.76) (diameter 0) (color 0 0 0 0)
   )
-  (junction (at 323.85 172.72) (diameter 0) (color 0 0 0 0)
-  )
   (junction (at 45.72 153.67) (diameter 0) (color 0 0 0 0)
   )
@@
     (stroke (width 0) (type default) (color 0 0 0 0))
   )
+  (wire (pts (xy 78.74 153.67) (xy 78.74 160.02))
+    (stroke (width 0) (type default) (color 0 0 0 0))
+  )
   (wire (pts (xy 248.92 144.78) (xy 284.48 144.78))
     (stroke (width 0) (type default) (color 0 0 0 0))
@@
     (stroke (width 0) (type default) (color 0 0 0 0))
   )
+  (wire (pts (xy 78.74 160.02) (xy 96.52 160.02))
+    (stroke (width 0) (type default) (color 0 0 0 0))
+  )
   (wire (pts (xy 60.96 125.73) (xy 60.96 132.08))
     (stroke (width 0) (type default) (color 0 0 0 0))
@@
     (stroke (width 0) (type default) (color 0 0 0 0))
   )
-  (wire (pts (xy 323.85 172.72) (xy 334.01 172.72))
-    (stroke (width 0) (type default) (color 0 0 0 0))
-  )
-  (wire (pts (xy 316.23 172.72) (xy 323.85 172.72))
+  (wire (pts (xy 316.23 172.72) (xy 334.01 172.72))
     (stroke (width 0) (type default) (color 0 0 0 0))
   )
@@
     (stroke (width 0) (type default) (color 0 0 0 0))
   )
-  (wire (pts (xy 292.1 173.99) (xy 341.63 173.99))
+  (wire (pts (xy 292.1 173.99) (xy 323.85 173.99))
     (stroke (width 0) (type default) (color 0 0 0 0))
   )
@@
     (stroke (width 0) (type default) (color 0 0 0 0))
   )
-  (wire (pts (xy 60.96 160.02) (xy 96.52 160.02))
+  (wire (pts (xy 60.96 160.02) (xy 78.74 160.02))
     (stroke (width 0) (type default) (color 0 0 0 0))
   )
@@
     (stroke (width 0) (type default) (color 0 0 0 0))
   )
-  (wire (pts (xy 323.85 167.64) (xy 323.85 172.72))
-    (stroke (width 0) (type default) (color 0 0 0 0))
-  )
   (wire (pts (xy 326.39 101.6) (xy 308.61 101.6))
     (stroke (width 0) (type default) (color 0 0 0 0))
@@
     (stroke (width 0) (type default) (color 0 0 0 0))
   )
+  (wire (pts (xy 323.85 173.99) (xy 341.63 173.99))
+    (stroke (width 0) (type default) (color 0 0 0 0))
+  )
   (wire (pts (xy 167.64 118.11) (xy 185.42 118.11))
     (stroke (width 0) (type default) (color 0 0 0 0))
@@
     (stroke (width 0) (type default) (color 0 0 0 0))
   )
+  (wire (pts (xy 323.85 167.64) (xy 323.85 173.99))
+    (stroke (width 0) (type default) (color 0 0 0 0))
+  )

Commit message: Update of schematic infos and backplate
Other:
- company: (none) -> Cipulot's PCB Design 
- title: (none) -> EC87
Changed lines of the file:
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@@
 (kicad_sch (version 20211123) (generator eeschema)
-  (paper "A3")
+  (paper "A4")
+  (title_block
+    (title "EC87")
+    (date "2022-03-30")
+    (rev "1")
+    (company "Cipulot's PCB Design ")
+  )
   (junction (at 266.7 116.84) (diameter 0) (color 0 0 0 0)
   )
