File: PCB/plate.kicad_pcb (KiCad board)
At the start: 2 copper layers, 354 x 121 mm, 127 parts, among them SW10 EC_SW, SW11 EC_SW, SW12 EC_SW, SW13 EC_SW, SW14 EC_SW, SW15 EC_SW, SW16 EC_SW, SW17 EC_SW, SW18 EC_SW, SW19 EC_SW, SW2 EC_SW, SW20 EC_SW, SW21 EC_SW, SW22 EC_SW, SW23 EC_SW, SW24 EC_SW, SW25 EC_SW, SW26 EC_SW, SW27 EC_SW, SW28 EC_SW, SW29 EC_SW, SW3 EC_SW, SW30 EC_SW, SW31 EC_SW, SW32 EC_SW, SW33 EC_SW, SW34 EC_SW, SW35 EC_SW, SW36 EC_SW, SW37 EC_SW, SW38 EC_SW, SW39 EC_SW, SW4 EC_SW, SW40 EC_SW, SW41 EC_SW, SW42 EC_SW, SW43 EC_SW, SW44 EC_SW, SW45 EC_SW, SW46 EC_SW, SW47 EC_SW, SW48 EC_SW, SW49 EC_SW, SW5 EC_SW, SW50 EC_SW, SW51 EC_SW, SW52 EC_SW, SW53 EC_SW, SW54 EC_SW, SW55 EC_SW, SW56 EC_SW, SW57 EC_SW, SW58 EC_SW, SW59 EC_SW, SW6 EC_SW, SW60 EC_SW, SW61 EC_SW, SW62 EC_SW, SW63 EC_SW, SW64 EC_SW, SW65 EC_SW, SW66 EC_SW, SW67 EC_SW, SW68 EC_SW, SW69 EC_SW, SW7 EC_SW, SW70 EC_SW, SW71 EC_SW, SW72 EC_SW, SW73 EC_SW, SW74 EC_SW, SW75 EC_SW, SW76 EC_SW, SW77 EC_SW, SW78 EC_SW, SW79 EC_SW, SW8 EC_SW, SW80 EC_SW, SW81 EC_SW, SW82 EC_SW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

Commit message: Update plate 2u holes
Other:
- board text added: "Topre"
Changed lines of the file:
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@@
       (effects (font (size 0.8 0.8) (thickness 0.12)))
     )
-    (fp_line (start -16.2 5.5) (end -13.601924 7) (layer "Edge.Cuts") (width 0.12))
-    (fp_line (start 16.2 5.5) (end 13.601924 7) (layer "Edge.Cuts") (width 0.12))
-    (fp_line (start 16.2 0) (end 16.2 5.5) (layer "Edge.Cuts") (width 0.12))
-    (fp_line (start -16.2 0) (end -16.2 -7) (layer "Edge.Cuts") (width 0.12))
-    (fp_line (start -16.2 0) (end -16.2 5.5) (layer "Edge.Cuts") (width 0.12))
-    (fp_line (start 16.2 -7) (end 16.2 0) (layer "Edge.Cuts") (width 0.12))
-    (fp_line (start 13.601924 7) (end -13.601924 7) (layer "Edge.Cuts") (width 0.12))
-    (fp_line (start -16.2 -7) (end 16.2 -7) (layer "Edge.Cuts") (width 0.12))
+    (fp_line (start 16 5.5) (end 13 7) (layer "Edge.Cuts") (width 0.12))
+    (fp_line (start 16 0) (end 16 5.5) (layer "Edge.Cuts") (width 0.12))
+    (fp_line (start 16 -7) (end 16 0) (layer "Edge.Cuts") (width 0.12))
+    (fp_line (start -16 0) (end -16 5.5) (layer "Edge.Cuts") (width 0.12))
+    (fp_line (start -16 0) (end -16 -7) (layer "Edge.Cuts") (width 0.12))
+    (fp_line (start 13 7) (end -13 7) (layer "Edge.Cuts") (width 0.12))
+    (fp_line (start -16 5.5) (end -13 7) (layer "Edge.Cuts") (width 0.12))
+    (fp_line (start -16 -7) (end 16 -7) (layer "Edge.Cuts") (width 0.12))
     (model "${KICAD6_3DMODEL_DIR}/cipulot_parts.3dshapes/Topre_Housing.step"
       (offset (xyz -9.3 -9.05 -5.25))
@@
       (effects (font (size 0.8 0.8) (thickness 0.12)))
     )
-    (fp_line (start 13.601924 7) (end -13.601924 7) (layer "Edge.Cuts") (width 0.12))
-    (fp_line (start 16.2 -7) (end 16.2 0) (layer "Edge.Cuts") (width 0.12))
-    (fp_line (start 16.2 0) (end 16.2 5.5) (layer "Edge.Cuts") (width 0.12))
-    (fp_line (start 16.2 5.5) (end 13.601924 7) (layer "Edge.Cuts") (width 0.12))
-    (fp_line (start -16.2 -7) (end 16.2 -7) (layer "Edge.Cuts") (width 0.12))
-    (fp_line (start -16.2 0) (end -16.2 5.5) (layer "Edge.Cuts") (width 0.12))
-    (fp_line (start -16.2 5.5) (end -13.601924 7) (layer "Edge.Cuts") (width 0.12))
-    (fp_line (start -16.2 0) (end -16.2 -7) (layer "Edge.Cuts") (width 0.12))
+    (fp_line (start -16 -7) (end 16 -7) (layer "Edge.Cuts") (width 0.12))
+    (fp_line (start 16 -7) (end 16 0) (layer "Edge.Cuts") (width 0.12))
+    (fp_line (start -16 5.5) (end -13 7) (layer "Edge.Cuts") (width 0.12))
+    (fp_line (start 16 5.5) (end 13 7) (layer "Edge.Cuts") (width 0.12))
+    (fp_line (start -16 0) (end -16 -7) (layer "Edge.Cuts") (width 0.12))
+    (fp_line (start -16 0) (end -16 5.5) (layer "Edge.Cuts") (width 0.12))
+    (fp_line (start 13 7) (end -13 7) (layer "Edge.Cuts") (width 0.12))
+    (fp_line (start 16 0) (end 16 5.5) (layer "Edge.Cuts") (width 0.12))
     (model "${KICAD6_3DMODEL_DIR}/cipulot_parts.3dshapes/Topre_Housing.step"
       (offset (xyz -9.3 -9.05 -5.25))
@@
       (effects (font (size 0.8 0.8) (thickness 0.12)))
     )
-    (fp_line (start -16.2 0) (end -16.2 5.5) (layer "Edge.Cuts") (width 0.12))
-    (fp_line (start -16.2 5.5) (end -13.601924 7) (layer "Edge.Cuts") (width 0.12))
-    (fp_line (start 13.601924 7) (end -13.601924 7) (layer "Edge.Cuts") (width 0.12))
-    (fp_line (start -16.2 -7) (end 16.2 -7) (layer "Edge.Cuts") (width 0.12))
-    (fp_line (start 16.2 5.5) (end 13.601924 7) (layer "Edge.Cuts") (width 0.12))
-    (fp_line (start 16.2 -7) (end 16.2 0) (layer "Edge.Cuts") (width 0.12))
-    (fp_line (start 16.2 0) (end 16.2 5.5) (layer "Edge.Cuts") (width 0.12))
-    (fp_line (start -16.2 0) (end -16.2 -7) (layer "Edge.Cuts") (width 0.12))
+    (fp_line (start -16 0) (end -16 5.5) (layer "Edge.Cuts") (width 0.12))
+    (fp_line (start -16 -7) (end 16 -7) (layer "Edge.Cuts") (width 0.12))
+    (fp_line (start 16 5.5) (end 13 7) (layer "Edge.Cuts") (width 0.12))
+    (fp_line (start 16 0) (end 16 5.5) (layer "Edge.Cuts") (width 0.12))
+    (fp_line (start -16 0) (end -16 -7) (layer "Edge.Cuts") (width 0.12))
+    (fp_line (start 13 7) (end -13 7) (layer "Edge.Cuts") (width 0.12))
+    (fp_line (start -16 5.5) (end -13 7) (layer "Edge.Cuts") (width 0.12))
+    (fp_line (start 16 -7) (end 16 0) (layer "Edge.Cuts") (width 0.12))
     (model "${KICAD6_3DMODEL_DIR}/cipulot_parts.3dshapes/Topre_Housing.step"
       (offset (xyz -9.3 -9.05 -5.25))
@@
       (effects (font (size 0.8 0.8) (thickness 0.12)))
     )
-    (fp_line (start -16.2 0) (end -16.2 5.5) (layer "Edge.Cuts") (width 0.12))
-    (fp_line (start -16.2 5.5) (end -13.601924 7) (layer "Edge.Cuts") (width 0.12))
-    (fp_line (start -16.2 0) (end -16.2 -7) (layer "Edge.Cuts") (width 0.12))
-    (fp_line (start -16.2 -7) (end 16.2 -7) (layer "Edge.Cuts") (width 0.12))
-    (fp_line (start 13.601924 7) (end -13.601924 7) (layer "Edge.Cuts") (width 0.12))
-    (fp_line (start 16.2 5.5) (end 13.601924 7) (layer "Edge.Cuts") (width 0.12))
-    (fp_line (start 16.2 -7) (end 16.2 0) (layer "Edge.Cuts") (width 0.12))
-    (fp_line (start 16.2 0) (end 16.2 5.5) (layer "Edge.Cuts") (width 0.12))
+    (fp_line (start -16 5.5) (end -13 7) (layer "Edge.Cuts") (width 0.12))
+    (fp_line (start -16 0) (end -16 5.5) (layer "Edge.Cuts") (width 0.12))
+    (fp_line (start -16 0) (end -16 -7) (layer "Edge.Cuts") (width 0.12))
+    (fp_line (start 16 5.5) (end 13 7) (layer "Edge.Cuts") (width 0.12))
+    (fp_line (start 16 -7) (end 16 0) (layer "Edge.Cuts") (width 0.12))
+    (fp_line (start 13 7) (end -13 7) (layer "Edge.Cuts") (width 0.12))
+    (fp_line (start 16 0) (end 16 5.5) (layer "Edge.Cuts") (width 0.12))
+    (fp_line (start -16 -7) (end 16 -7) (layer "Edge.Cuts") (width 0.12))
     (model "${KICAD6_3DMODEL_DIR}/cipulot_parts.3dshapes/Topre_Housing.step"
       (offset (xyz -9.3 -9.05 -5.25))
@@
   (gr_line (start 329.2425 84.3375) (end 338.6425 84.3375) (layer "User.2") (width 0.1))
   (gr_line (start 314.83 84.3375) (end 324.23 84.3375) (layer "User.2") (width 0.1))
+  (gr_text "Topre" (at 379.67 202.18) (layer "B.SilkS")
+    (effects (font (size 1.5 1.5) (thickness 0.3) italic) (justify mirror))
+  )
   (gr_text "SWDIO\n" (at 340.41 153.21 90) (layer "F.SilkS")
     (effects (font (size 1 1) (thickness 0.15)) (justify right))
