File: PCB/Rev 1/plate.kicad_pcb (KiCad board)
At the start: 2 copper layers, 354 x 121 mm, 127 parts, among them SW10 EC_SW, SW11 EC_SW, SW12 EC_SW, SW13 EC_SW, SW14 EC_SW, SW15 EC_SW, SW16 EC_SW, SW17 EC_SW, SW18 EC_SW, SW19 EC_SW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

Commit message: Update to remove logo
Parts:
- removed the G*** at (376.4, 155.2)
